File: Flight controller 1.0.0.kicad_pcb (KiCad board)
At the start: 4 copper layers, 36 x 36 mm, 68 parts, among them J1 USB_C_Receptacle_USB2.0_14P, J2 Conn_01x08_Socket, J3 Conn_01x04_Pin, J4 Conn_01x04, J5 Conn_01x04, SW1 SW_Push, Y1 Crystal_GND24

Commit message: Povecane komponente
Parts:
- removed C20: 22u, Capacitor_SMD:C_0201_0603Metric
- C12, C13, C24: value 0.1u -> 100n
- C14, C6: footprint Capacitor_SMD:C_0201_0603Metric -> Capacitor_SMD:C_0402_1005Metric
- C15: value 1u -> 10u; footprint Capacitor_SMD:C_0201_0603Metric -> Capacitor_SMD:C_0402_1005Metric
- C21: value 47u -> 4.7u; footprint Capacitor_SMD:C_0201_0603Metric -> Capacitor_SMD:C_0402_1005Metric
- C23: value 1u -> 100n
- C26: footprint Capacitor_SMD:C_0201_0603Metric -> Capacitor_SMD:C_0603_1608Metric
- L1: value 2.5u -> 10u; footprint Inductor_SMD:L_0603_1608Metric -> Inductor_SMD:L_0805_2012Metric
- R10: value 18.2k -> 110k
- moved C25 1.33 mm to (146.5, 121.0), turned to 90 degrees
- moved C21 1.03 mm to (134.5, 122.2)
- moved C26 0.75 mm to (144.2, 122.0)
- moved C15 0.47 mm to (154.0, 113.1)
- moved L1 0.45 mm to (143.8, 125.1)
- moved R12 0.41 mm to (144.2, 120.2)
- moved R11 0.35 mm to (144.2, 118.3)
- moved C23 0.31 mm to (145.2, 123.5)
- moved C24 0.31 mm to (143.4, 123.5)
- moved C2 0.30 mm to (137.3, 98.5)
- moved C6 0.24 mm to (137.4, 99.5)
- moved C13 0.24 mm to (154.0, 115.0)
- moved R7 0.15 mm to (152.2, 114.1)
- moved R13 0.15 mm to (147.3, 124.8)
- moved C14 0.10 mm to (154.0, 111.0)
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Routing:
- net Net-(U2-FB): track 7.26 -> 8.64 mm
- net GND: track 65.5 -> 64.5 mm, vias 65 -> 64
- net +3.3V: track 127.3 -> 128.2 mm
- net +5V_BUCK: track 71.5 -> 72.0 mm
- net Net-(U2-BST): track 8.94 -> 8.44 mm

Commit message: Kondenzatori-povecani
Parts:
- C1, C10, C11, C12, C13, C16, C17, C18, C19, C2, C22, C23, C24, C25, C3, C4, C5, C7, C8, C9: footprint Capacitor_SMD:C_0201_0603Metric -> Capacitor_SMD:C_0402_1005Metric
- moved R9 0.83 mm to (147.2, 111.1)
- moved D4 0.83 mm to (147.2, 112.9)
- moved C9 0.73 mm to (135.5, 104.2)
- moved R1 0.62 mm to (152.0, 116.9)
- moved C26 0.55 mm to (144.2, 121.5)
- moved D3 0.54 mm to (148.2, 116.9)
- moved C24 0.53 mm to (143.0, 123.1)
- moved C19 0.48 mm to (134.7, 105.8)
- moved C12 0.43 mm to (144.5, 112.2)
- moved FB1 0.40 mm to (133.1, 106.6)
- moved C23 0.40 mm to (145.4, 123.1)
- moved C5 0.38 mm to (146.9, 99.1)
- moved D1 0.38 mm to (150.4, 97.8)
- moved C10 0.37 mm to (143.0, 113.9)
- moved C17 0.35 mm to (135.9, 105.8)
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Routing:
- net +3.3V: track 128.2 -> 125.4 mm
- net /LED_STM32: track 19.7 -> 20.7 mm
- net Net-(U2-BST): track 8.44 -> 7.72 mm
- net Net-(D8-A): track 8.33 -> 8.96 mm
- net /BOOT0: track 40.7 -> 41.3 mm
- net Net-(D3-A): track 4.36 -> 4.94 mm
- net /VDDA: track 5.03 -> 5.60 mm

Commit message: ispocetka
Parts:
- U1: renamed from STM32; footprint Package_QFP:LQFP-64_7x7mm_P0.4mm -> Package_QFP:LQFP-64_10x10mm_P0.5mm
- renumbered BUCK to U2, LDO to U3
