File: Flight controller 1.0.0.kicad_sch (KiCad schematic)
At the start: 67 parts, among them J1 USB_C_Receptacle_USB2.0_14P, J2 Conn_01x08_Socket, J3 Conn_01x04_Pin, J4 Conn_01x04, J5 Conn_01x04, Q1 NPN, SW1 SW_Push, U1 STM32F405RGT6, U2 LT8610, U3 LT1117-ADJ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

Commit message: Povecane komponente
Parts:
- removed C20: 22u, Capacitor_SMD:C_0201_0603Metric, symbol Device:C
- C14, C6: footprint Capacitor_SMD:C_0201_0603Metric -> Capacitor_SMD:C_0402_1005Metric; LCSC (none) -> C315248
- C15: value 1u -> 10u; footprint Capacitor_SMD:C_0201_0603Metric -> Capacitor_SMD:C_0402_1005Metric; LCSC C53067 -> C315248
- C21: value 47u -> 4.7u; footprint Capacitor_SMD:C_0201_0603Metric -> Capacitor_SMD:C_0402_1005Metric; LCSC (none) -> C6119795
- C26: footprint Capacitor_SMD:C_0201_0603Metric -> Capacitor_SMD:C_0603_1608Metric; LCSC (none) -> C178330
- D1, D2: LCSC (none) -> C5345968
- D3, D4, D5: LCSC (none) -> C19273151
- D6: LCSC (none) -> C49207092
- D7: LCSC (none) -> C30584800; now left out of the parts list
- D8: LCSC (none) -> C30584800
- FB1: LCSC (none) -> C107335
- J1: LCSC (none) -> C165948
- J2: LCSC (none) -> C265120
- J3, J4, J5, Q1, TP1, TP2, TP3: now left out of the parts list
- L1: value 2.5u -> 10u; footprint Inductor_SMD:L_0603_1608Metric -> Inductor_SMD:L_0805_2012Metric; LCSC (none) -> C53436344
- MT1: LCSC (none) -> C3288646
- R1, R4: LCSC (none) -> C98220
- R10: value 18.2k -> 110k; LCSC (none) -> C2906984
- R11: LCSC (none) -> C137764
- R12: LCSC (none) -> C2907115
- R13, R7, R9: LCSC (none) -> C2907148
- R14: LCSC (none) -> C2907113; now left out of the parts list
- R15: LCSC (none) -> C98220; now left out of the parts list
- R2, R3: LCSC (none) -> C2907044
- R5: LCSC (none) -> C25804
- R6: LCSC (none) -> C2933134
- R8: LCSC (none) -> C2907113
- SW1: LCSC (none) -> C2886902
- U1: LCSC (none) -> C15742
- U2: LCSC (none) -> C462619
- U3: LCSC (none) -> C3014296
- Y1: LCSC (none) -> C2916927
Other:
- moved on the sheet: C21

Commit message: Kondenzatori-povecani
Parts:
- C1, C12, C13, C17, C2, C23, C24, C3, C4, C5, C9: footprint Capacitor_SMD:C_0201_0603Metric -> Capacitor_SMD:C_0402_1005Metric; LCSC C49062 -> C60474
- C10, C19, C22: footprint Capacitor_SMD:C_0201_0603Metric -> Capacitor_SMD:C_0402_1005Metric; LCSC C76941 -> C60133
- C11, C7, C8: footprint Capacitor_SMD:C_0201_0603Metric -> Capacitor_SMD:C_0402_1005Metric; LCSC C318539 -> C170151
- C16, C18, C25: footprint Capacitor_SMD:C_0201_0603Metric -> Capacitor_SMD:C_0402_1005Metric; LCSC C43535 -> C713505
Changed lines of the file:
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@@
 			)
 		)
-		(property "Footprint" "Capacitor_SMD:C_0201_0603Metric"
+		(property "Footprint" "Capacitor_SMD:C_0402_1005Metric"
 			(at 176.2252 90.17 0)
 			(effects
@@
 			)
 		)
-		(property "LCSC" "C49062"
+		(property "LCSC" "C60474"
 			(at 175.26 86.36 0)
 			(effects
@@
 			)
 		)
-		(property "Footprint" "Capacitor_SMD:C_0201_0603Metric"
+		(property "Footprint" "Capacitor_SMD:C_0402_1005Metric"
 			(at 23.8252 265.43 0)
 			(effects
@@
 			)
 		)
-		(property "LCSC" "C49062"
+		(property "LCSC" "C60474"
 			(at 22.86 261.62 0)
 			(effects
@@
 			)
 		)
-		(property "Footprint" "Capacitor_SMD:C_0201_0603Metric"
+		(property "Footprint" "Capacitor_SMD:C_0402_1005Metric"
 			(at 177.8 164.1348 0)
 			(effects
@@
 			)
 		)
-		(property "LCSC" "C318539"
+		(property "LCSC" "C170151"
 			(at 173.99 165.1 90)
 			(effects
@@
 			)
 		)
-		(property "Footprint" "Capacitor_SMD:C_0201_0603Metric"
+		(property "Footprint" "Capacitor_SMD:C_0402_1005Metric"
 			(at 219.4052 88.9 0)
 			(effects
@@
 			)
 		)
-		(property "LCSC" "C76941"
+		(property "LCSC" "C60133"
 			(at 218.44 85.09 0)
 			(effects
@@
 			)
 		)
-		(property "Footprint" "Capacitor_SMD:C_0201_0603Metric"
+		(property "Footprint" "Capacitor_SMD:C_0402_1005Metric"
 			(at 129.2352 111.76 0)
 			(effects
@@
 			)
 		)
-		(property "LCSC" "C49062"
+		(property "LCSC" "C60474"
 			(at 128.27 107.95 0)
 			(effects
@@
 			)
 		)
-		(property "Footprint" "Capacitor_SMD:C_0201_0603Metric"
+		(property "Footprint" "Capacitor_SMD:C_0402_1005Metric"
 			(at 359.7148 21.59 0)
 			(effects
@@
 			)
 		)
-		(property "LCSC" "C49062"
+		(property "LCSC" "C60474"
 			(at 360.68 25.4 0)
 			(effects
@@
 			)
 		)
-		(property "Footprint" "Capacitor_SMD:C_0201_0603Metric"
+		(property "Footprint" "Capacitor_SMD:C_0402_1005Metric"
 			(at 338.1248 194.31 0)
 			(effects
@@
 			)
 		)
-		(property "LCSC" "C49062"
+		(property "LCSC" "C60474"
 			(at 339.09 198.12 0)
 			(effects
@@
 			)
 		)
-		(property "Footprint" "Capacitor_SMD:C_0201_0603Metric"
+		(property "Footprint" "Capacitor_SMD:C_0402_1005Metric"
 			(at 292.1 206.0448 0)
 			(effects
@@
 			)
 		)
-		(property "LCSC" "C76941"
+		(property "LCSC" "C60133"
 			(at 288.29 207.01 90)
 			(effects
@@
 			)
 		)
-		(property "Footprint" "Capacitor_SMD:C_0201_0603Metric"
+		(property "Footprint" "Capacitor_SMD:C_0402_1005Metric"
 			(at 153.67 134.9248 0)
 			(effects
@@
 			)
 		)
-		(property "LCSC" "C43535"
+		(property "LCSC" "C713505"
 			(at 149.86 135.89 90)
 			(effects
@@
 			)
 		)
-		(property "Footprint" "Capacitor_SMD:C_0201_0603Metric"
+		(property "Footprint" "Capacitor_SMD:C_0402_1005Metric"
 			(at 330.5048 184.15 0)
 			(effects
@@
 			)
 		)
-		(property "LCSC" "C49062"
+		(property "LCSC" "C60474"
 			(at 331.47 187.96 0)
 			(effects
@@
 			)
 		)
-		(property "Footprint" "Capacitor_SMD:C_0201_0603Metric"
+		(property "Footprint" "Capacitor_SMD:C_0402_1005Metric"
 			(at 187.6552 90.17 0)
 			(effects
@@
 			)
 		)
-		(property "LCSC" "C49062"
+		(property "LCSC" "C60474"
 			(at 186.69 86.36 0)
 			(effects
@@
 			)
 		)
-		(property "Footprint" "Capacitor_SMD:C_0201_0603Metric"
+		(property "Footprint" "Capacitor_SMD:C_0402_1005Metric"
 			(at 371.1448 21.59 0)
 			(effects
@@
 			)
 		)
-		(property "LCSC" "C318539"
+		(property "LCSC" "C170151"
 			(at 372.11 25.4 0)
 			(effects
@@
 			)
 		)
-		(property "Footprint" "Capacitor_SMD:C_0201_0603Metric"
+		(property "Footprint" "Capacitor_SMD:C_0402_1005Metric"
 			(at 153.3652 90.17 0)
 			(effects
@@
 			)
 		)
-		(property "LCSC" "C49062"
+		(property "LCSC" "C60474"
 			(at 152.4 86.36 0)
 			(effects
@@
 			)
 		)
-		(property "Footprint" "Capacitor_SMD:C_0201_0603Metric"
+		(property "Footprint" "Capacitor_SMD:C_0402_1005Metric"
 			(at 164.7952 90.17 0)
 			(effects
@@
 			)
 		)
-		(property "LCSC" "C49062"
+		(property "LCSC" "C60474"
 			(at 163.83 86.36 0)
 			(effects
@@
 			)
 		)
-		(property "Footprint" "Capacitor_SMD:C_0201_0603Metric"
+		(property "Footprint" "Capacitor_SMD:C_0402_1005Metric"
 			(at 232.1052 88.9 0)
 			(effects
@@
 			)
 		)
-		(property "LCSC" "C49062"
+		(property "LCSC" "C60474"
 			(at 231.14 85.09 0)
 			(effects
@@
 			)
 		)
-		(property "Footprint" "Capacitor_SMD:C_0201_0603Metric"
+		(property "Footprint" "Capacitor_SMD:C_0402_1005Metric"
 			(at 141.9352 90.17 0)
 			(effects
@@
 			)
 		)
-		(property "LCSC" "C49062"
+		(property "LCSC" "C60474"
 			(at 140.97 86.36 0)
 			(effects
@@
 			)
 		)
-		(property "Footprint" "Capacitor_SMD:C_0201_0603Metric"
+		(property "Footprint" "Capacitor_SMD:C_0402_1005Metric"
 			(at 382.5748 21.59 0)
 			(effects
@@
 			)
 		)
-		(property "LCSC" "C76941"
+		(property "LCSC" "C60133"
 			(at 383.54 25.4 0)
 			(effects
@@
 			)
 		)
-		(property "Footprint" "Capacitor_SMD:C_0201_0603Metric"
+		(property "Footprint" "Capacitor_SMD:C_0402_1005Metric"
 			(at 142.5448 120.65 0)
 			(effects
@@
 			)
 		)
-		(property "LCSC" "C43535"
+		(property "LCSC" "C713505"
 			(at 143.51 124.46 0)
 			(effects
@@
 			)
 		)
-		(property "Footprint" "Capacitor_SMD:C_0201_0603Metric"
+		(property "Footprint" "Capacitor_SMD:C_0402_1005Metric"
 			(at 177.8 170.4848 0)
 			(effects
@@
 			)
 		)
-		(property "LCSC" "C318539"
+		(property "LCSC" "C170151"
 			(at 173.99 171.45 90)
 			(effects
@@
 			)
 		)
-		(property "Footprint" "Capacitor_SMD:C_0201_0603Metric"
+		(property "Footprint" "Capacitor_SMD:C_0402_1005Metric"
 			(at 353.06 213.6648 0)
 			(effects
@@
 			)
 		)
-		(property "LCSC" "C43535"
+		(property "LCSC" "C713505"
 			(at 349.25 214.63 90)
 			(effects

Commit message: ispocetka
Parts:
- U1: footprint Package_QFP:LQFP-64_7x7mm_P0.4mm -> Package_QFP:LQFP-64_10x10mm_P0.5mm
Changed lines of the file:
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@@
 			)
 		)
-		(property "Footprint" "Package_QFP:LQFP-64_7x7mm_P0.4mm"
+		(property "Footprint" "Package_QFP:LQFP-64_10x10mm_P0.5mm"
 			(at 189.23 185.42 0)
 			(effects
